File: keyboard/scheme/keyboard/keyboard.kicad_sch (KiCad schematic)
At the start: 37 parts, among them SW10 SW_DIP_x01, SW11 SW_DIP_x01, SW12 SW_DIP_x01, SW13 SW_DIP_x01, SW14 SW_DIP_x01, SW15 SW_DIP_x01, SW16 SW_DIP_x01, SW17 SW_DIP_x01, SW18 SW_DIP_x01, SW19 SW_DIP_x01, SW2 SW_DIP_x01, SW20 SW_DIP_x01, SW21 SW_DIP_x01, SW22 SW_DIP_x01, SW23 SW_DIP_x01, SW24 SW_DIP_x01, SW25 SW_DIP_x01, SW26 SW_DIP_x01, SW27 SW_DIP_x01, SW28 SW_DIP_x01, SW29 SW_DIP_x01, SW3 SW_DIP_x01, SW30 SW_DIP_x01, SW31 SW_DIP_x01, SW32 SW_DIP_x01, SW33 SW_DIP_x01, SW34 SW_DIP_x01, SW35 SW_DIP_x01, SW36 SW_DIP_x01, SW4 SW_DIP_x01, SW5 SW_DIP_x01, SW7 SW_DIP_x01, SW8 SW_DIP_x01, SW9 SW_DIP_x01

Commit message: Add power supply to keyboard scheme
Parts:
- added C1, C2, C3, C4: (no value), symbol Device:C
- added J1: (no value), symbol Connector_Generic:Conn_01x03
- added U2: (no value), symbol Regulator_Linear:AMS1117CD-3.3
- SW1, SW6: value (none) -> SW_DIP_x01; footprint (none) -> my_lib:btn_8x8
- U1: value (none) -> STM32F030F4Px; footprint (none) -> Package_SO:TSSOP-20_4.4x6.5mm_P0.65mm
Connections:
- net uart_tx: now also J1.3 (Pin_3)
- net GND: now reaches U1.15 (VSS)
- net GND: now also C1.2, C2.2, C3.2, C4.2, J1.2 (Pin_2), U2.1 (GND)
- net 3.3v: now reaches U1.16 (VDD)
- net 3.3v: now also U1.5 (VDDA), C1.1, C3.1, C4.1, U2.2 (VO)
- new net 5v: C2.1, J1.1 (Pin_1), U2.3 (VI)
